File: LHRCustomScreen/LHRCustomScreen.kicad_pcb (KiCad board)
At the start: 4 copper layers, 121 x 75 mm, 108 parts, among them J1 Conn_01x40, J2 Conn_02x02_Odd_Even, J3 Conn_01x02, J7 Conn_02x03_Odd_Even, Q1 CSD15571Q2, Q2 CSD15571Q2, Q3 CSD17571Q2, Q4 CSD17571Q2, SW1 SW_Push, U1 TPS62933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

Commit message: added 12v plane
added 12v plane
Parts:
- moved Cf1 2.80 mm to (103.5, 96.9)
- moved Rf1 2.80 mm to (100.3, 96.9)
- moved Ruvb1 1.75 mm to (89.5, 93.0)
Routing:
- net +12V: track 198.7 -> 70.5 mm, vias 2 -> 3
- net CSG: track 179.3 -> 171.0 mm
- net Net-(U4-EN_UVLO): track 72.1 -> 67.2 mm, vias 2 -> 0
- net Net-(U4-VIN): track 53.4 -> 49.0 mm, vias 0 -> 1
- net Change_Screen: track 88.6 -> 86.2 mm
- net Net-(U4-VISNS): track 66.1 -> 64.3 mm, vias 2 -> 1
- net Net-(Df1-K): track 3.49 -> 4.75 mm
- net SW2: track 47.3 -> 46.3 mm
- net Net-(U4-MODE): track 17.3 -> 16.5 mm
- net SWO: track 99.0 -> 98.1 mm
- net (no net): track 6.27 -> 5.62 mm
- added copper zone on B.Cu, net +12V
